Commit message: gazebo almost ok

File: fredo1/gazebo/urdf/fredo1.xacro (robot description, xacro)
@@ -7,4 +7,5 @@
   <xacro:include filename="$(find fredo1_robot)/urdf/links/link1.xacro"/>
   <xacro:include filename="$(find fredo1_robot)/urdf/links/link2.xacro"/>
+  <xacro:include filename="$(find fredo1_robot)/urdf/links/link3.xacro"/>
   <!-- <xacro:include filename="$(find fredo1_robot)/urdf/links/end_effector.xacro"/> -->
   <!-- Load joints -->
@@ -12,5 +13,5 @@
   <xacro:include filename="$(find fredo1_robot)/urdf/joints/joint1.xacro"/>
   <xacro:include filename="$(find fredo1_robot)/urdf/joints/joint2.xacro"/>
-  <!-- <xacro:include filename="$(find fredo1_robot)/urdf/joints/joint3.xacro"/> -->
+  <xacro:include filename="$(find fredo1_robot)/urdf/joints/joint3.xacro"/>
   <gazebo>
     <plugin name="gazebo_ros_control" filename="libgazebo_ros_control.so">

File: fredo1/gazebo/urdf/joints/joint0.xacro (robot description, xacro)
@@ -4,5 +4,5 @@
     <parent link="world"/>
     <child link="base_link"/>
-    <origin xyz="0 0 0.1" rpy="0 0 0"/>
+    <origin xyz="0 0 0.01" rpy="0 0 0"/>
   </joint>
 </robot>

File: fredo1/gazebo/urdf/joints/joint1.xacro (robot description, xacro)
@@ -4,5 +4,5 @@
     <parent link="base_link"/>
     <child link="link1"/>
-    <origin xyz="0 0 0.25" rpy="0 0 0"/>
+    <origin xyz="0.01916 -0.05981 0.06072" rpy="0 0 0"/>
     <axis xyz="0 0 1"/>
     <limit effort="10" velocity="1.0" lower="-1.57" upper="1.57"/>

File: fredo1/gazebo/urdf/joints/joint3.xacro (robot description, xacro)
@@ -2,9 +2,9 @@
 <robot xmlns:xacro="http://ros.org/wiki/xacro">
   <!-- Define the revolute joint -->
-  <joint name="joint2" type="revolute">
-    <parent link="link1"/>  <!-- Parent link is link1 -->
-    <child link="link2"/>   <!-- Child link is link2 -->
+  <joint name="joint3" type="revolute">
+    <parent link="link2"/>  <!-- Parent link is link1 -->
+    <child link="link3"/>   <!-- Child link is link2 -->
     <!-- Joint Origin -->
-    <origin xyz="-0.0299 -0.0105 0.0335" rpy="0 0 0"/> <!-- Position along Y axis of link1 -->
+    <origin xyz="0.0014 -0.01042 0.096" rpy="0 0 0"/> <!-- Position along Y axis of link1 -->
     <!-- Axis of Rotation: Y-axis -->
     <axis xyz="1 0 0"/>  <!-- Revolving around Y-axis -->
@@ -12,10 +12,10 @@
     <limit lower="-1.57" upper="1.57" effort="5" velocity="1"/>
   </joint>
-  <transmission name="joint2_trans">
+  <transmission name="joint3_trans">
     <type>transmission_interface/SimpleTransmission</type>
-    <joint name="joint2">
+    <joint name="joint3">
       <hardwareInterface>EffortJointInterface</hardwareInterface>
     </joint>
-    <actuator name="joint2_motor">
+    <actuator name="joint3_motor">
       <mechanicalReduction>1</mechanicalReduction>
     </actuator>

File: fredo1/gazebo/urdf/links/base_link.xacro (robot description, xacro)
@@ -1,5 +1,5 @@
 <?xml version="1.0"?>
 <robot xmlns:xacro="http://ros.org/wiki/xacro">
-  <!-- Define the Dummy World Link -->
+  <!-- Define the fredo1 World Link -->
   <link name="world"/>
   <!-- Base Link -->
@@ -7,14 +7,66 @@
     <!-- Visual -->
     <visual>
-      <origin xyz="0 0 0" rpy="0 0 0"/>
+      <origin xyz="0 0 0" rpy="1.5708 0 0"/>
       <geometry>
-        <box size="0.3 0.3 0.1"/>
+        <mesh filename="package://fredo1_robot/../cad/all_files/a_base.STL" scale="0.001 0.001 0.001"/>
       </geometry>
     </visual>
     <!-- Collision -->
     <collision>
-      <origin xyz="0 0 0" rpy="0 0 0"/>
+      <origin xyz="0 0 0" rpy="1.5708 0 0"/>
       <geometry>
-        <box size="0.3 0.3 0.1"/>
+        <mesh filename="package://fredo1_robot/../cad/all_files/a_base.STL" scale="0.001 0.001 0.001"/>
+      </geometry>
+    </collision>
+    <visual>
+      <origin xyz="0 0 0" rpy="1.5708 0 0"/>
+      <geometry>
+        <mesh filename="package://fredo1_robot/../cad/all_files/a_servo_1.STL" scale="0.001 0.001 0.001"/>
+      </geometry>
+    </visual>
+    <!-- Collision -->
+    <collision>
+      <origin xyz="0 0 0" rpy="1.5708 0 0"/>
+      <geometry>
+        <mesh filename="package://fredo1_robot/../cad/all_files/a_servo_1.STL" scale="0.001 0.001 0.001"/>
+      </geometry>
+    </collision>
+    <visual>
+      <origin xyz="0 0 0" rpy="1.5708 0 0"/>
+      <geometry>
+        <mesh filename="package://fredo1_robot/../cad/all_files/a_servo_2.STL" scale="0.001 0.001 0.001"/>
+      </geometry>
+    </visual>
+    <!-- Collision -->
+    <collision>
+      <origin xyz="0 0 0" rpy="1.5708 0 0"/>
+      <geometry>
+        <mesh filename="package://fredo1_robot/../cad/all_files/a_servo_2.STL" scale="0.001 0.001 0.001"/>
+      </geometry>
+    </collision>
+    <visual>
+      <origin xyz="0 0 0" rpy="1.5708 0 0"/>
+      <geometry>
+        <mesh filename="package://fredo1_robot/../cad/all_files/a_servo_3.STL" scale="0.001 0.001 0.001"/>
+      </geometry>
+    </visual>
+    <!-- Collision -->
+    <collision>
+      <origin xyz="0 0 0" rpy="1.5708 0 0"/>
+      <geometry>
+        <mesh filename="package://fredo1_robot/../cad/all_files/a_servo_3.STL" scale="0.001 0.001 0.001"/>
+      </geometry>
+    </collision>
+    <visual>
+      <origin xyz="0 0 0" rpy="1.5708 0 0"/>
+      <geometry>
+        <mesh filename="package://fredo1_robot/../cad/all_files/a_servo_4.STL" scale="0.001 0.001 0.001"/>
+      </geometry>
+    </visual>
+    <!-- Collision -->
+    <collision>
+      <origin xyz="0 0 0" rpy="1.5708 0 0"/>
+      <geometry>
+        <mesh filename="package://fredo1_robot/../cad/all_files/a_servo_4.STL" scale="0.001 0.001 0.001"/>
       </geometry>
     </collision>
@@ -35,5 +87,5 @@
   <!-- GAZEBO-specific Color -->
   <gazebo reference="base_link">
-    <material>Gazebo/Red</material>
+    <material>Gazebo/Gray</material>
     <static>false</static>
   </gazebo>

File: fredo1/gazebo/urdf/links/link1.xacro (robot description, xacro)
@@ -2,12 +2,100 @@
 <robot xmlns:xacro="http://ros.org/wiki/xacro">
   <link name="link1">
+    <!-- Visual -->
     <visual>
+      <origin xyz="-0.01916 0.05981 -0.06072" rpy="1.5708 0 0"/>
       <geometry>
-        <cylinder length="0.5" radius="0.05"/>
+        <mesh filename="package://fredo1_robot/../cad/all_files/b_servoarm.STL" scale="0.001 0.001 0.001"/>
       </geometry>
     </visual>
+    <!-- Collision -->
     <collision>
+      <origin xyz="-0.01916 0.05981 -0.06072" rpy="1.5708 0 0"/>
       <geometry>
-        <cylinder length="0.5" radius="0.05"/>
+        <mesh filename="package://fredo1_robot/../cad/all_files/b_servoarm.STL" scale="0.001 0.001 0.001"/>
+      </geometry>
+    </collision>
+    <!-- Visual -->
+    <visual>
+      <origin xyz="-0.01916 0.05981 -0.06072" rpy="1.5708 0 0"/>
+      <geometry>
+        <mesh filename="package://fredo1_robot/../cad/all_files/b_firstarm.STL" scale="0.001 0.001 0.001"/>
+      </geometry>
+    </visual>
+    <!-- Collision -->
+    <collision>
+      <origin xyz="-0.01916 0.05981 -0.06072" rpy="1.5708 0 0"/>
+      <geometry>
+        <mesh filename="package://fredo1_robot/../cad/all_files/b_firstarm.STL" scale="0.001 0.001 0.001"/>
+      </geometry>
+    </collision>
+    <!-- Visual -->
+    <visual>
+      <origin xyz="-0.01916 0.05981 -0.06072" rpy="1.5708 0 0"/>
+      <geometry>
+        <mesh filename="package://fredo1_robot/../cad/all_files/b_servo_1.STL" scale="0.001 0.001 0.001"/>
+      </geometry>
+    </visual>
+    <!-- Collision -->
+    <collision>
+      <origin xyz="-0.01916 0.05981 -0.06072" rpy="1.5708 0 0"/>
+      <geometry>
+        <mesh filename="package://fredo1_robot/../cad/all_files/b_servo_1.STL" scale="0.001 0.001 0.001"/>
+      </geometry>
+    </collision>
+    <!-- Visual -->
+    <visual>
+      <origin xyz="-0.01916 0.05981 -0.06072" rpy="1.5708 0 0"/>
+      <geometry>
+        <mesh filename="package://fredo1_robot/../cad/all_files/b_servo_2.STL" scale="0.001 0.001 0.001"/>
+      </geometry>
+    </visual>
+    <!-- Collision -->
+    <collision>
+      <origin xyz="-0.01916 0.05981 -0.06072" rpy="1.5708 0 0"/>
+      <geometry>
+        <mesh filename="package://fredo1_robot/../cad/all_files/b_servo_2.STL" scale="0.001 0.001 0.001"/>
+      </geometry>
+    </collision>
+    <!-- Visual -->
+    <visual>
+      <origin xyz="-0.01916 0.05981 -0.06072" rpy="1.5708 0 0"/>
+      <geometry>
+        <mesh filename="package://fredo1_robot/../cad/all_files/b_servo_3.STL" scale="0.001 0.001 0.001"/>
+      </geometry>
+    </visual>
+    <!-- Collision -->
+    <collision>
+      <origin xyz="-0.01916 0.05981 -0.06072" rpy="1.5708 0 0"/>
+      <geometry>
+        <mesh filename="package://fredo1_robot/../cad/all_files/b_servo_3.STL" scale="0.001 0.001 0.001"/>
+      </geometry>
+    </collision>
+    <!-- Visual -->
+    <visual>
+      <origin xyz="-0.01916 0.05981 -0.06072" rpy="1.5708 0 0"/>
+      <geometry>
+        <mesh filename="package://fredo1_robot/../cad/all_files/b_rod.STL" scale="0.001 0.001 0.001"/>
+      </geometry>
+    </visual>
+    <!-- Collision -->
+    <collision>
+      <origin xyz="-0.01916 0.05981 -0.06072" rpy="1.5708 0 0"/>
+      <geometry>
+        <mesh filename="package://fredo1_robot/../cad/all_files/b_rod.STL" scale="0.001 0.001 0.001"/>
+      </geometry>
+    </collision>
+    <!-- Visual -->
+    <visual>
+      <origin xyz="-0.01916 0.05981 -0.06072" rpy="1.5708 0 0"/>
+      <geometry>
+        <mesh filename="package://fredo1_robot/../cad/all_files/b_servo_4.STL" scale="0.001 0.001 0.001"/>
+      </geometry>
+    </visual>
+    <!-- Collision -->
+    <collision>
+      <origin xyz="-0.01916 0.05981 -0.06072" rpy="1.5708 0 0"/>
+      <geometry>
+        <mesh filename="package://fredo1_robot/../cad/all_files/b_servo_4.STL" scale="0.001 0.001 0.001"/>
       </geometry>
     </collision>

File: fredo1/gazebo/urdf/links/link2.xacro (robot description, xacro)
@@ -5,20 +5,117 @@
     <!-- Visual -->
     <visual>
-      <origin xyz="0 0 0.25" rpy="0 0 0"/>
+      <origin xyz="0.01074 0.07031 -0.09422" rpy="1.5708 0 0"/>
       <geometry>
-        <cylinder length="0.5" radius="0.05"/>
+        <mesh filename="package://fredo1_robot/../cad/all_files/c_servoarm.STL" scale="0.001 0.001 0.001"/>
       </geometry>
-      <material name="Green"/>
     </visual>
     <!-- Collision -->
     <collision>
-      <origin xyz="0 0 0.25" rpy="0 0 0"/>
+      <origin xyz="0.01074 0.07031 -0.09422" rpy="1.5708 0 0"/>
       <geometry>
-        <cylinder length="0.5" radius="0.05"/>
+        <mesh filename="package://fredo1_robot/../cad/all_files/c_servoarm.STL" scale="0.001 0.001 0.001"/>
+      </geometry>
+    </collision>
+    <!-- Visual -->
+    <visual>
+      <origin xyz="0.01074 0.07031 -0.09422" rpy="1.5708 0 0"/>
+      <geometry>
+        <mesh filename="package://fredo1_robot/../cad/all_files/c_secondarm.STL" scale="0.001 0.001 0.001"/>
+      </geometry>
+    </visual>
+    <!-- Collision -->
+    <collision>
+      <origin xyz="0.01074 0.07031 -0.09422" rpy="1.5708 0 0"/>
+      <geometry>
+        <mesh filename="package://fredo1_robot/../cad/all_files/c_secondarm.STL" scale="0.001 0.001 0.001"/>
+      </geometry>
+    </collision>
+    <!-- Visual -->
+    <visual>
+      <origin xyz="0.01074 0.07031 -0.09422" rpy="1.5708 0 0"/>
+      <geometry>
+        <mesh filename="package://fredo1_robot/../cad/all_files/c_servo_1.STL" scale="0.001 0.001 0.001"/>
+      </geometry>
+    </visual>
+    <!-- Collision -->
+    <collision>
+      <origin xyz="0.01074 0.07031 -0.09422" rpy="1.5708 0 0"/>
+      <geometry>
+        <mesh filename="package://fredo1_robot/../cad/all_files/c_servo_1.STL" scale="0.001 0.001 0.001"/>
+      </geometry>
+    </collision>
+    <!-- Visual -->
+    <visual>
+      <origin xyz="0.01074 0.07031 -0.09422" rpy="1.5708 0 0"/>
+      <geometry>
+        <mesh filename="package://fredo1_robot/../cad/all_files/c_servo_2.STL" scale="0.001 0.001 0.001"/>
+      </geometry>
+    </visual>
+    <!-- Collision -->
+    <collision>
+      <origin xyz="0.01074 0.07031 -0.09422" rpy="1.5708 0 0"/>
+      <geometry>
+        <mesh filename="package://fredo1_robot/../cad/all_files/c_servo_2.STL" scale="0.001 0.001 0.001"/>
+      </geometry>
+    </collision>
+    <!-- Visual -->
+    <visual>
+      <origin xyz="0.01074 0.07031 -0.09422" rpy="1.5708 0 0"/>
+      <geometry>
+        <mesh filename="package://fredo1_robot/../cad/all_files/c_servo_3.STL" scale="0.001 0.001 0.001"/>
+      </geometry>
+    </visual>
+    <!-- Collision -->
+    <collision>
+      <origin xyz="0.01074 0.07031 -0.09422" rpy="1.5708 0 0"/>
+      <geometry>
+        <mesh filename="package://fredo1_robot/../cad/all_files/c_servo_3.STL" scale="0.001 0.001 0.001"/>
+      </geometry>
+    </collision>
+    <!-- Visual -->
+    <visual>
+      <origin xyz="0.01074 0.07031 -0.09422" rpy="1.5708 0 0"/>
+      <geometry>
+        <mesh filename="package://fredo1_robot/../cad/all_files/c_servoplate.STL" scale="0.001 0.001 0.001"/>
+      </geometry>
+    </visual>
+    <!-- Collision -->
+    <collision>
+      <origin xyz="0.01074 0.07031 -0.09422" rpy="1.5708 0 0"/>
+      <geometry>
+        <mesh filename="package://fredo1_robot/../cad/all_files/c_servoplate.STL" scale="0.001 0.001 0.001"/>
+      </geometry>
+    </collision>
+    <!-- Visual -->
+    <visual>
+      <origin xyz="0.01074 0.07031 -0.09422" rpy="1.5708 0 0"/>
+      <geometry>
+        <mesh filename="package://fredo1_robot/../cad/all_files/c_rod.STL" scale="0.001 0.001 0.001"/>
+      </geometry>
+    </visual>
+    <!-- Collision -->
+    <collision>
+      <origin xyz="0.01074 0.07031 -0.09422" rpy="1.5708 0 0"/>
+      <geometry>
+        <mesh filename="package://fredo1_robot/../cad/all_files/c_rod.STL" scale="0.001 0.001 0.001"/>
+      </geometry>
+    </collision>
+    <!-- Visual -->
+    <visual>
+      <origin xyz="0.01074 0.07031 -0.09422" rpy="1.5708 0 0"/>
+      <geometry>
+        <mesh filename="package://fredo1_robot/../cad/all_files/c_servo_4.STL" scale="0.001 0.001 0.001"/>
+      </geometry>
+    </visual>
+    <!-- Collision -->
+    <collision>
+      <origin xyz="0.01074 0.07031 -0.09422" rpy="1.5708 0 0"/>
+      <geometry>
+        <mesh filename="package://fredo1_robot/../cad/all_files/c_servo_4.STL" scale="0.001 0.001 0.001"/>
       </geometry>
     </collision>
     <!-- Inertial -->
     <inertial>
-      <mass value="1.0"/>
+      <mass value="0.01"/>
       <inertia ixx="0.005" ixy="0.0" ixz="0.0"
                iyy="0.005" iyz="0.0"

File: fredo1/gazebo/urdf/materials.xacro (robot description, xacro)
@@ -10,3 +10,6 @@
     <color rgba="0 1 0 1"/>
   </material>
+  <material name="Gray">
+    <color rgba="1.0 1.0 1.0 1"/>
+  </material>
 </robot>
