Commit message: gazebo confirmed

File: fredo1/gazebo/urdf/joints/joint3.xacro (robot description, xacro)
@@ -6,5 +6,5 @@
     <child link="link3"/>   <!-- Child link is link2 -->
     <!-- Joint Origin -->
-    <origin xyz="0.0014 -0.01042 0.096" rpy="0 0 0"/> <!-- Position along Y axis of link1 -->
+    <origin xyz="-0.0014 -0.01042 0.096" rpy="0 0 0"/> <!-- Position along Y axis of link1 -->
     <!-- Axis of Rotation: Y-axis -->
     <axis xyz="1 0 0"/>  <!-- Revolving around Y-axis -->

File: fredo1/gazebo/urdf/links/link2.xacro (robot description, xacro)
@@ -117,5 +117,5 @@
     <!-- Inertial -->
     <inertial>
-      <mass value="0.01"/>
+      <mass value="0.1"/>
       <inertia ixx="0.005" ixy="0.0" ixz="0.0"
                iyy="0.005" iyz="0.0"

File: fredo1/gazebo/urdf/links/link3.xacro (robot description, xacro)
@@ -20,11 +20,11 @@
     <!-- Inertial -->
     <inertial>
-      <mass value="0.00100001"/>
-      <inertia ixx="0.00" ixy="0.0" ixz="0.0"
-               iyy="0.00" iyz="0.0"
-               izz="0.00"/>
+      <mass value="0.1"/>
+      <inertia ixx="0.005" ixy="0.0" ixz="0.0"
+               iyy="0.005" iyz="0.0"
+               izz="0.005"/>
     </inertial>
   </link>
-  <gazebo reference="link1">
+  <gazebo reference="link3">
     <material>Gazebo/Red</material>
   </gazebo>
