Commit message: gazebo + ros + rviz => consolidated

File: fredo1/gazebo/urdf/joints/joint0.xacro (robot description, xacro)
@@ -5,4 +5,14 @@
     <child link="base_link"/>
     <origin xyz="0 0 0.01" rpy="0 0 0"/>
+    <limit effort="10" velocity="1.0" lower="0" upper="0"/>
   </joint>
+  <!-- <transmission name="joint0_trans">
+    <type>transmission_interface/SimpleTransmission</type>
+    <joint name="joint0">
+      <hardwareInterface>EffortJointInterface</hardwareInterface>
+    </joint>
+    <actuator name="joint0_motor">
+      <mechanicalReduction>1</mechanicalReduction>
+    </actuator>
+  </transmission> -->
 </robot>
