Commit message: bullet okay

File: dummy/bullet/urdf/dummy.urdf (robot description, URDF)
Before this commit: robot dummy, 4 links, 3 joints
Links:
- removed link link3
- link base: mass 2.0 -> 0.1; geometry collision box size=0.3 0.3 0.1; visual box size=0.3 0.3 0.1
- link link1: mass 1.0 -> 0.1; geometry collision cylinder length=0.5 radius=0.05; visual cylinder length=0.5 radius=0.05
- link link2: mass 1.0 -> 0.1; geometry collision cylinder length=0.5 radius=0.05; visual cylinder length=0.5 radius=0.05
Joints:
- removed joint joint_3
- joint joint_1: origin xyz=0.1916 -0.5981 0.6072 rpy=0 0 0 -> xyz=0 0 0.1 rpy=0 0 0
- joint joint_2: origin xyz=-0.299 -0.105 0.335 rpy=0 0 0 -> xyz=0 0 0.5 rpy=0 0 0
