Commit message: add fredo1 firmware

File: fredo1/bullet/urdf/fredo1.urdf (robot description, URDF)
Before this commit: robot fredo1, 4 links, 3 joints
Links:
- link base: mass 2.0 -> 0.1
- link link1: mass 1.0 -> 0.1
- link link2: mass 1.0 -> 0.1
- link link3: mass 1.0 -> 0.1
Joints:
- joint joint_1: limit lower=-3.14159 upper=3.14159 effort=1 velocity=1 -> lower=-1.39626 upper=3.14159 effort=1 velocity=1
- joint joint_2: limit lower=-3.14159 upper=3.14159 effort=1 velocity=1 -> lower=-1.48352 upper=1.57079 effort=1 velocity=1
- joint joint_3: limit lower=-3.14159 upper=3.14159 effort=1 velocity=1 -> lower=-1.48352 upper=1.57079 effort=1 velocity=1
